Commit message: feat(ros2): realistic Gazebo runs with friction in the physics
The Gazebo path now runs with the environment profile, by default
config/imperfections/realistic.yaml (launch and controller), plus a
`seed` launch argument (default: the profile's seed).

- sim.launch.py writes the profile's friction (coulomb_nm,
  viscous_nm_s_rad) into the xacro args joint_<i>_friction and
  joint_<i>_damping, i.e. each arm joint's <dynamics>, so the physics
  engine applies it instead of a torque from the measured velocity.
- The controller gives ImperfectJointInterface the profile with
  friction zeroed, emulates model mismatch by perturbing its own model,
  rejects payload_kg != 0 and warns once that timing jitter is ignored.
- tools/run_e2e.py passes the scenario seed; new scenario E2E-09
  (Gazebo, realistic, seed 7, E2E-02 thresholds).
- README "Environment configuration", conventions pointer and an
  ADR-011 update.

File: sim/urdf/cobot30_5.urdf.xacro (robot description, xacro)
@@ -4,8 +4,25 @@
      cobot30_5_gazebo.urdf is generated from cobot30_5.urdf by tools/fix_urdf_inertia.py
      (gazebo_urdf): Gazebo has no joint armature, so each joint's reflected rotor inertia is
-     added to its child link as a rotor disc about the joint axis (an approximation, see there). -->
+     added to its child link as a rotor disc about the joint axis (an approximation, see there).
+     joint_<i>_friction (Coulomb, N m) and joint_<i>_damping (viscous, N m s/rad) set each arm
+     joint's <dynamics>; sim.launch.py fills them from the imperfection profile's friction, so
+     the physics engine applies it (default 0: no joint friction). -->
 <robot xmlns:xacro="http://www.ros.org/wiki/xacro" name="cobot30_5">
   <xacro:arg name="controllers_yaml" default=""/>
   <xacro:arg name="home_q" default="0.0 0.5235987755982988 0.0 -1.5707963267948966 0.0 1.0471975511965976 0.0"/>
+  <xacro:arg name="joint_1_friction" default="0.0"/>
+  <xacro:arg name="joint_1_damping" default="0.0"/>
+  <xacro:arg name="joint_2_friction" default="0.0"/>
+  <xacro:arg name="joint_2_damping" default="0.0"/>
+  <xacro:arg name="joint_3_friction" default="0.0"/>
+  <xacro:arg name="joint_3_damping" default="0.0"/>
+  <xacro:arg name="joint_4_friction" default="0.0"/>
+  <xacro:arg name="joint_4_damping" default="0.0"/>
+  <xacro:arg name="joint_5_friction" default="0.0"/>
+  <xacro:arg name="joint_5_damping" default="0.0"/>
+  <xacro:arg name="joint_6_friction" default="0.0"/>
+  <xacro:arg name="joint_6_damping" default="0.0"/>
+  <xacro:arg name="joint_7_friction" default="0.0"/>
+  <xacro:arg name="joint_7_damping" default="0.0"/>
   <xacro:include filename="cobot30_5_gazebo.urdf"/>
   <xacro:property name="home" value="${'$(arg home_q)'.split()}"/>
